Commit message: model can show on rviz

File: install/lab1_1/share/lab1_1/descriptions/robot.urdf (robot description, URDF)
Before this commit: robot robot, 1 links, 0 joints
Links:
- added link steer_front_left; visual cylinder length=0.001 radius=0.01
- added link steer_front_right; visual cylinder length=0.001 radius=0.01
- added link wheel_front_left; visual mesh filename=package://lab1_1/meshes/limo_optimal_wheels.dae scale=1 1 1
- added link wheel_front_right; visual mesh filename=package://lab1_1/meshes/limo_optimal_wheels.dae scale=1 1 1
- added link wheel_rear_left; visual mesh filename=package://lab1_1/meshes/limo_optimal_wheels.dae scale=1 1 1
- added link wheel_rear_right; visual mesh filename=package://lab1_1/meshes/limo_optimal_wheels.dae scale=1 1 1
- link base: mass 1.0 -> 3.0; geometry collision mesh filename=package://lab1_1/meshes/limo_optimal.dae scale=1 1 1; visual mesh filename=package://lab1_1/meshes/limo_optimal.dae scale=1 1 1
Joints:
- added joint joint_wheel_rear_left: type continuous, parent base, child wheel_rear_left, origin xyz=-0.1 0.065 0.045 rpy=0 0 0, axis 0 1 0
- added joint joint_wheel_rear_right: type continuous, parent base, child wheel_rear_right, origin xyz=-0.1 -0.065 0.045 rpy=0 0 3.14, axis 0 1 0
- added joint rotation_joint_front_left: type continuous, parent steer_front_left, child wheel_front_left, origin xyz=0 0 0 rpy=0 0 3.14, axis 0 1 0
- added joint rotation_joint_front_right: type continuous, parent steer_front_right, child wheel_front_right, origin xyz=0 0 0 rpy=0 0 3.14, axis 0 1 0
- added joint steering_joint_front_left: type revolute, parent base, child steer_front_left, origin xyz=0.1 0.065 0.045 rpy=0 0 3.14, axis 0 0 1, limit lower=-0.5 upper=0.5 effort=10.0 velocity=1.0
- added joint steering_joint_front_right: type revolute, parent base, child steer_front_right, origin xyz=0.1 -0.065 0.045 rpy=0 0 0, axis 0 0 1, limit lower=-0.5 upper=0.5 effort=10.0 velocity=1.0

File: src/lab1_1/descriptions/robot.urdf (robot description, URDF)
Before this commit: robot robot, 2 links, 1 joints
Links:
- removed link link1
- added link steer_front_left; visual cylinder length=0.001 radius=0.01
- added link steer_front_right; visual cylinder length=0.001 radius=0.01
- added link wheel_front_left; visual mesh filename=package://lab1_1/meshes/limo_optimal_wheels.dae scale=1 1 1
- added link wheel_front_right; visual mesh filename=package://lab1_1/meshes/limo_optimal_wheels.dae scale=1 1 1
- added link wheel_rear_left; visual mesh filename=package://lab1_1/meshes/limo_optimal_wheels.dae scale=1 1 1
- added link wheel_rear_right; visual mesh filename=package://lab1_1/meshes/limo_optimal_wheels.dae scale=1 1 1
- link base: mass 1.0 -> 3.0; geometry collision mesh filename=package://lab1_1/meshes/limo_optimal.dae scale=1 1 1; visual mesh filename=package://lab1_1/meshes/limo_optimal.dae scale=1 1 1
Joints:
- removed joint base_to_link1
- added joint joint_wheel_rear_left: type continuous, parent base, child wheel_rear_left, origin xyz=-0.1 0.065 0.045 rpy=0 0 0, axis 0 1 0
- added joint joint_wheel_rear_right: type continuous, parent base, child wheel_rear_right, origin xyz=-0.1 -0.065 0.045 rpy=0 0 3.14, axis 0 1 0
- added joint rotation_joint_front_left: type continuous, parent steer_front_left, child wheel_front_left, origin xyz=0 0 0 rpy=0 0 3.14, axis 0 1 0
- added joint rotation_joint_front_right: type continuous, parent steer_front_right, child wheel_front_right, origin xyz=0 0 0 rpy=0 0 3.14, axis 0 1 0
- added joint steering_joint_front_left: type revolute, parent base, child steer_front_left, origin xyz=0.1 0.065 0.045 rpy=0 0 3.14, axis 0 0 1, limit lower=-0.5 upper=0.5 effort=10.0 velocity=1.0
- added joint steering_joint_front_right: type revolute, parent base, child steer_front_right, origin xyz=0.1 -0.065 0.045 rpy=0 0 0, axis 0 0 1, limit lower=-0.5 upper=0.5 effort=10.0 velocity=1.0

Commit message: .

File: install/lab1_1/share/lab1_1/descriptions/robot.urdf (robot description, URDF)
Before this commit: robot robot_with_ackermann, 7 links, 6 joints
Links:
- link steer_front_left: mass None -> 0.2; geometry 
- link steer_front_right: mass None -> 0.2; geometry 
- link wheel_front_left: mass None -> 0.2; geometry collision mesh filename=package://lab1_1/meshes/limo_optimal_wheels.dae scale=1 1 1; visual mesh filename=package://lab1_1/meshes/limo_optimal_wheels.dae scale=1 1 1
- link wheel_front_right: mass None -> 0.2; geometry collision mesh filename=package://lab1_1/meshes/limo_optimal_wheels.dae scale=1 1 1; visual mesh filename=package://lab1_1/meshes/limo_optimal_wheels.dae scale=1 1 1
- link wheel_rear_left: mass None -> 0.2; geometry collision mesh filename=package://lab1_1/meshes/limo_optimal_wheels.dae scale=1 1 1; visual mesh filename=package://lab1_1/meshes/limo_optimal_wheels.dae scale=1 1 1
- link wheel_rear_right: mass None -> 0.2; geometry collision mesh filename=package://lab1_1/meshes/limo_optimal_wheels.dae scale=1 1 1; visual mesh filename=package://lab1_1/meshes/limo_optimal_wheels.dae scale=1 1 1
